File: GBA_EMU.sch (EAGLE design)
At the start: 62 parts, among them Q1 MOSFET-PCHANNEL, SW1 LEFT, SW2 RIGHT, SW3 PWR_SWITCH, U1 RPI-ZERO, U2 FT230X, U3 MCP1642B-ADJ, U4 LM4875, U5 V_REG_LDOSMD2, U6 MIC7221, U7 AZV321, X1 LINK_SOCKET, X2 HEADPHONE

Commit message: Update GBA_EMU.sch
Parts:
- R9: value 309k -> 430k
Changed lines of the file:
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@@
 <part name="L4" library="rcl" deviceset="L-EU" device="WE-TPC" value="4.7uH"/>
 <part name="R7" library="rcl" deviceset="R-EU_" device="R0805" value="976k"/>
-<part name="R9" library="rcl" deviceset="R-EU_" device="R0805" value="309k"/>
+<part name="R9" library="rcl" deviceset="R-EU_" device="R0805" value="430k"/>
 <part name="GND13" library="SparkFun-Aesthetics" deviceset="GND" device=""/>
 <part name="GND14" library="SparkFun-Aesthetics" deviceset="GND" device=""/>
